File: gnss_board.kicad_pcb (KiCad board)
At the start: 2 copper layers, 0 parts

Commit message: Add footprints and arange components around
Parts:
- added C1: 1nF, Capacitor_SMD:C_1206_3216Metric, F.Cu at (53.6, 70.4)
- added C10: 2.2uF, Capacitor_SMD:C_0805_2012Metric, F.Cu at (81.9, 100.6)
- added C11: 100nF, Capacitor_SMD:C_0805_2012Metric, F.Cu at (81.9, 103.6)
- added C12: 22uF, Capacitor_SMD:C_0805_2012Metric, F.Cu at (77.2, 97.6)
- added C13: 100nF, Capacitor_SMD:C_0805_2012Metric, F.Cu at (77.2, 100.6)
- added C14: 100nF, Capacitor_SMD:C_0805_2012Metric, F.Cu at (77.2, 103.6)
- added C16: 12pF, Capacitor_SMD:C_0805_2012Metric, F.Cu at (97.8, 82.2)
- added C17: 470uF, Capacitor_THT:CP_Radial_D6.3mm_P2.50mm, F.Cu at (90.4, 92.5)
- added C18: 100nF, Capacitor_SMD:C_0805_2012Metric, F.Cu at (97.8, 85.3)
- added C19: 220pF, Capacitor_SMD:C_0805_2012Metric, F.Cu at (97.8, 88.3)
- added C2: 1nF, Capacitor_SMD:C_1206_3216Metric, F.Cu at (52.4, 85.8)
- added C3: 1nF, Capacitor_SMD:C_1206_3216Metric, F.Cu at (52.4, 89.1)
- added C4: 1nF, Capacitor_SMD:C_1206_3216Metric, F.Cu at (52.4, 92.5)
- added C6: 10uF, Capacitor_SMD:C_0805_2012Metric, F.Cu at (89.1, 108.4)
- added C7: 15uF, Capacitor_THT:CP_Radial_D6.3mm_P2.50mm, F.Cu at (90.4, 84.7)
- added C8: 22uF, Capacitor_SMD:C_0805_2012Metric, F.Cu at (108.2, 71.3)
- added C9: 100nF, Capacitor_SMD:C_0805_2012Metric, F.Cu at (81.9, 97.6)
- added D1: MB10S, GNSS Board:SOIC245P670X290-4N, F.Cu at (60.3, 85.2)
- added D2: MB10S, gnss_board:SOIC245P670X290-4N, F.Cu at (60.3, 91.7)
- added D6: LED, LED_SMD:LED_0805_2012Metric, F.Cu at (97.8, 91.3)
- added J1: Conn_01x10_Pin, Connector_JST:JST_SH_BM10B-SRSS-TB_1x10-1MP_P1.00mm_Vertical, F.Cu at (65.7, 73.8)
- added L1: FB0805, Inductor_SMD:L_0805_2012Metric_Pad1.15x1.40mm_HandSolder, F.Cu at (108.3, 68.4)
- added L2: 33uH, gnss_board:INDPM120120X800N, F.Cu at (77.6, 73.8)
- added R1: 75R, Resistor_SMD:R_0805_2012Metric, F.Cu at (52.9, 73.5)
- added R10: 2.2K, Resistor_SMD:R_0805_2012Metric, F.Cu at (87.2, 71.3)
- added R11: 12.1K, Resistor_SMD:R_0805_2012Metric, F.Cu at (87.2, 74.3)
- added R12: 2.2K, Resistor_SMD:R_0805_2012Metric, F.Cu at (89.1, 99.5)
- added R13: 2.2K, Resistor_SMD:R_0805_2012Metric, F.Cu at (89.1, 102.5)
- added R14: 2.2K, Resistor_SMD:R_0805_2012Metric, F.Cu at (89.1, 105.4)
- added R15: 2.2K, Resistor_SMD:R_0805_2012Metric, F.Cu at (93.5, 99.5)
- added R16: 2.2K, Resistor_SMD:R_0805_2012Metric, F.Cu at (93.5, 102.5)
- added R17: 2.2K, Resistor_SMD:R_0805_2012Metric, F.Cu at (93.5, 105.4)
- added R18: 2.2K, Resistor_SMD:R_0805_2012Metric, F.Cu at (97.9, 99.5)
- added R19: 2.2K, Resistor_SMD:R_0805_2012Metric, F.Cu at (97.9, 102.5)
- added R2: 75R, Resistor_SMD:R_0805_2012Metric, F.Cu at (52.9, 76.5)
- added R20: 10K, Resistor_SMD:R_0805_2012Metric, F.Cu at (97.9, 105.4)
- added R21: 4.42K, Resistor_SMD:R_0805_2012Metric, F.Cu at (91.6, 68.4)
- added R22: 180K, Resistor_SMD:R_0805_2012Metric, F.Cu at (91.6, 71.3)
- added R24: 0.03R, Resistor_SMD:R_1206_3216Metric, F.Cu at (73.0, 93.7)
- added R25: 4.7K, Resistor_SMD:R_2512_6332Metric, F.Cu at (74.5, 89.6)
- added R28: 301K, Resistor_SMD:R_0805_2012Metric, F.Cu at (91.6, 74.3)
- added R29: 95.3K, Resistor_SMD:R_0805_2012Metric, F.Cu at (96.0, 68.4)
- added R3: 75R, Resistor_SMD:R_0805_2012Metric, F.Cu at (48.1, 72.2)
- added R30: 4.7R, Resistor_SMD:R_0805_2012Metric, F.Cu at (96.0, 71.3)
- added R31: 22R, Resistor_SMD:R_0805_2012Metric, F.Cu at (96.0, 74.3)
- added R4: 75R, Resistor_SMD:R_0805_2012Metric, F.Cu at (48.1, 75.2)
- added R5: 49.9R, Resistor_SMD:R_0805_2012Metric, F.Cu at (103.7, 68.4)
- added R6: 49.9R, Resistor_SMD:R_0805_2012Metric, F.Cu at (103.7, 71.3)
- added R7: 49.9R, Resistor_SMD:R_0805_2012Metric, F.Cu at (103.7, 74.3)
- added R8: 49.9R, Resistor_SMD:R_0805_2012Metric, F.Cu at (103.7, 77.2)
- added R9: 2.2K, Resistor_SMD:R_0805_2012Metric, F.Cu at (87.2, 68.4)
- added TVS1: ESDS314DBVR(SOT-23-5), Package_TO_SOT_SMD:SOT-23-5, F.Cu at (87.6, 78.1)
- added TVS2: D_TVS, Diode_SMD:D_0603_1608Metric, F.Cu at (108.4, 75.9)
- added TVS3: D_TVS, Diode_SMD:D_0603_1608Metric, F.Cu at (108.4, 78.5)
- added U1: H1102NL, GNSS Board:H11X_PUL, F.Cu at (67.2, 103.8)
- added U2: LAN8710A, Package_DFN_QFN:QFN-32-1EP_5x5mm_P0.5mm_EP3.3x3.3mm_ThermalVias, F.Cu at (82.8, 91.0)
- added U3: TPS2375D, GNSS Board:SOIC127P599X175-8N, F.Cu at (74.9, 84.0)
- added U4: TX4138(ESOIC-8), Package_SO:SOIC-8-1EP_3.9x4.9mm_P1.27mm_EP2.29x3mm_ThermalVias, F.Cu at (83.3, 84.1)
