File: gnss_board.kicad_sch (KiCad schematic)
At the start: 79 parts, among them J1 Conn_01x10_Pin, J2 Serial Connector, Q1 BC817, Q2 BC817, T1 LMUN2211LT1G, U1 H1102NL, U2 LAN8710A, U3 TPS2375D, U4 TX4138(ESOIC-8), U5 ESP32-WROOM-32E, U6 UM980

Commit message: Add GNSS module as well
Parts:
- added BT1: 6.8mm, SparkFun-Battery:ML414H_IV01E, symbol SparkFun-Battery:Battery_6.8mm_ML414H_IV01E
- added C23, C25: 100pF, Capacitor_SMD:C_0805_2012Metric, symbol Device:C_Small
- added C24: 0.1uF, Capacitor_SMD:C_0805_2012Metric, symbol Device:C_Small
- added C26: 2.2uF, Capacitor_SMD:C_0805_2012Metric, symbol Device:C_Small
- added C27: 100nF, Capacitor_SMD:C_0805_2012Metric, symbol Device:C_Small
- added C28: 1uF, Capacitor_SMD:C_0805_2012Metric, symbol Device:C_Small
- added D10: PMEG4005EJ, SparkFun-Semiconductor-Standard:SOD-323, symbol SparkFun-DiscreteSemi:D_Schottky_0.5A_40V_0.42V
- added D11: PESD0805, Capacitor_SMD:C_0805_2012Metric, symbol SparkFun-DiscreteSemi:D_TVS_0402
- added D12: PESD3V3L4UG, SparkFun-Semiconductor-Standard:SOT-353, symbol SparkFun-DiscreteSemi:D_TVS_ESD_4
- added D4: Red, SparkFun-LED:LED_0603_1608Metric_Red, symbol SparkFun-LED:LED_Red_0603
- added D7: Yellow, SparkFun-LED:LED_0603_1608Metric_Yellow, symbol SparkFun-LED:LED_Yellow_0603
- added D8: Blue, SparkFun-LED:LED_0603_1608Metric_Blue, symbol SparkFun-LED:LED_Blue_0603
- added D9: White, SparkFun-LED:LED_0603_1608Metric_White, symbol SparkFun-LED:LED_White_0603
- added J3: U.FL, SparkFun-Connector:U.FL, symbol SparkFun-RF:U.FL
- added J4: Conn_01x04_Pin, Connector_PinHeader_2.54mm:PinHeader_1x04_P2.54mm_Vertical, symbol Connector:Conn_01x04_Pin
- added L3: 68nH, Inductor_SMD:L_0805_2012Metric_Pad1.05x1.20mm_HandSolder, symbol SparkFun-Coil:68nH_0402_0.2A
- added R37, R39, R53: 10K, Resistor_SMD:R_0805_2012Metric, symbol Device:R
- added R38, R40, R41, R42, R43, R44, R45, R46, R47, R48, R49, R50, R51, R52: 33R, Resistor_SMD:R_0805_2012Metric, symbol Device:R
- added R57, R58, R61: 1K, Resistor_SMD:R_0805_2012Metric, symbol Device:R
- added R59, R60: 2.2K, Resistor_SMD:R_0805_2012Metric, symbol Device:R
- added TP1, TP2: PTH, SparkFun-Connector:1x01, symbol SparkFun-Connector:TestPoint_PTH
Connections:
- net VCC is gone; now on net +3.3V: U6.33 (VCC), U6.34 (VCC)
- net +3.3V: now also C26.2, C27.2, D10.A, J4.1 (Pin_1), R37.2, R39.2, R53.2, R58.1
- net GND: now also BT1.-, C24.2, C25.2, C26.1, C27.1, C28.1, D11.1 (A1), D12.2 (A), D4.1 (K), D7.1 (K), D8.1 (K), D9.1 (K), J3.2 (Ext), J4.4 (Pin_4)
- net GNSS_TXD1: now reaches U5.13 (IO14)
- net GNSS_TXD1: now also R40.2
- net GNSS_RXD1: now reaches U5.23 (IO15)
- net GNSS_RXD1: now also R41.2
- net GNSS_TXD2: now reaches U5.6 (IO34)
- net GNSS_TXD2: now also R42.2
- net GNSS_RXD2: now reaches U5.7 (IO35)
- net GNSS_RXD2: now also R43.2
- net at U6.19 (PVT_STAT): now also R48.1
- net at U6.2 (ANT_IN): now also C23.2
- net at U6.20 (RTK_STAT): now also R47.1
- net at U6.21 (ERR_STAT): now also R46.1
- net at U6.26 (RXD2): now also R43.1
- net at U6.27 (TXD2): now also R42.1
- net at U6.28 (BIF_28): now also R51.2
- net at U6.29 (BIF_29): now also R52.2
- net at U6.30 (TXD3): now also R44.1
- net at U6.31 (RXD3): now also R45.1
- net GNSS_V_BCKP: now reaches U6.36 (V_BCKP)
- net GNSS_V_BCKP: now also BT1.+, C28.2, R57.1
- net at U6.42 (TXD1): now also R40.1
- net at U6.43 (RXD1): now also R41.1
- net at U6.49 (~{RESET}): now also R38.2
- net at U6.51 (EVENT): now also R50.1
- net at U6.53 (PPS): now also R49.1
- net at U6.7 (VCC_RF): now also C24.1, C25.1, L3.1
- new net: R37.1, R52.1, TP1.1
- new net: C23.1, D11.2 (A2), J3.1 (In), L3.2
- new net: D4.2 (A), R58.2
- new net: D8.2 (A), R60.2
- new net: D7.2 (A), R59.2
- new net: R39.1, R51.1, TP2.1
- new net: D10.C, R57.2
- new net: D9.2 (A), R61.2
- new net GNSS_ERR_STAT: R46.2
- new net GNSS_EVENT: R50.2
- new net GNSS_PPS: R49.2, R59.1
- new net GNSS_PVT_STAT: R48.2, R60.1
- new net GNSS_RTK_STAT: R47.2, R61.1
- new net GNSS_RXD3: D12.3 (K2), J4.3 (Pin_3), R45.2
- new net GNSS_TXD3: D12.1 (K1), J4.2 (Pin_2), R44.2
- new net ~{GNSS_RESET}: R38.1, R53.1
- no-connect marks 12 -> 36
Other:
- note added: "GNSS Serial Connector"
- note added: "LEDs"
- note added: "UM980 GNSS"
- moved on the sheet: J2, Q1, Q2, R34, R35

Commit message: Messing around
Parts:
- D12: footprint SparkFun-Semiconductor-Standard:SOT-353 -> Package_TO_SOT_SMD:SOT-353_SC-70-5_Handsoldering; PROD_ID DIO-19494 -> (none)
Connections:
- net ESP_RXD0: now also D12.4 (K3)
- net ESP_TXD0: now also D12.5 (K4)
- no-connect marks 36 -> 34
Changed lines of the file:
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@@
 	)
 	(no_connect
-		(at 341.63 234.95)
-	)
-	(no_connect
 		(at 365.76 111.76)
 	)
@@
 	)
 	(no_connect
-		(at 344.17 234.95)
-	)
-	(no_connect
 		(at 233.68 190.5)
 	)
@@
 	(wire
 		(pts
+			(xy 341.63 234.95) (xy 341.63 233.68)
+		)
+		(stroke
+			(width 0)
+			(type default)
+		)
+	)
+	(wire
+		(pts
 			(xy 339.09 232.41) (xy 339.09 234.95)
 		)
@@
 	(wire
 		(pts
+			(xy 347.98 234.95) (xy 347.98 237.49)
+		)
+		(stroke
+			(width 0)
+			(type default)
+		)
+	)
+	(wire
+		(pts
 			(xy 109.22 223.52) (xy 121.92 223.52)
 		)
@@
 	(wire
 		(pts
+			(xy 349.25 233.68) (xy 349.25 234.95)
+		)
+		(stroke
+			(width 0)
+			(type default)
+		)
+	)
+	(wire
+		(pts
 			(xy 46.99 50.8) (xy 46.99 68.58)
 		)
@@
 	(wire
 		(pts
+			(xy 349.25 234.95) (xy 353.06 234.95)
+		)
+		(stroke
+			(width 0)
+			(type default)
+		)
+	)
+	(wire
+		(pts
 			(xy 248.92 106.68) (xy 252.73 106.68)
 		)
@@
 	(wire
 		(pts
+			(xy 344.17 234.95) (xy 347.98 234.95)
+		)
+		(stroke
+			(width 0)
+			(type default)
+		)
+	)
+	(wire
+		(pts
 			(xy 31.75 64.77) (xy 58.42 64.77)
 		)
@@
 	(wire
 		(pts
+			(xy 347.98 237.49) (xy 353.06 237.49)
+		)
+		(stroke
+			(width 0)
+			(type default)
+		)
+	)
+	(wire
+		(pts
 			(xy 214.63 207.01) (xy 214.63 208.28)
 		)
@@
 	(wire
 		(pts
+			(xy 341.63 233.68) (xy 349.25 233.68)
+		)
+		(stroke
+			(width 0)
+			(type default)
+		)
+	)
+	(wire
+		(pts
 			(xy 109.22 226.06) (xy 121.92 226.06)
 		)
@@
 		)
 	)
+	(global_label "ESP_RXD0"
+		(shape input)
+		(at 353.06 234.95 0)
+		(fields_autoplaced yes)
+		(effects
+			(font
+				(size 1.27 1.27)
+			)
+			(justify left)
+		)
+		(property "Intersheetrefs" "${INTERSHEET_REFS}"
+			(at 365.6003 234.95 0)
+			(effects
+				(font
+					(size 1.27 1.27)
+				)
+				(justify left)
+				(hide yes)
+			)
+		)
+	)
 	(global_label "GNSS_RXD2"
 		(shape input)
@@
 		)
 	)
+	(global_label "ESP_TXD0"
+		(shape input)
+		(at 353.06 237.49 0)
+		(fields_autoplaced yes)
+		(effects
+			(font
+				(size 1.27 1.27)
+			)
+			(justify left)
+		)
+		(property "Intersheetrefs" "${INTERSHEET_REFS}"
+			(at 365.2979 237.49 0)
+			(effects
+				(font
+					(size 1.27 1.27)
+				)
+				(justify left)
+				(hide yes)
+			)
+		)
+	)
 	(global_label "ETH_PHY_PWR"
 		(shape input)
@@
 			)
 		)
-		(property "Footprint" "SparkFun-Semiconductor-Standard:SOT-353"
+		(property "Footprint" "Package_TO_SOT_SMD:SOT-353_SC-70-5_Handsoldering"
 			(at 339.09 248.92 0)
 			(effects
@@
 			(effects
 				(font
-					(size 1.27 1.27)
-				)
-				(hide yes)
-			)
-		)
-		(property "PROD_ID" "DIO-19494"
-			(at 339.09 254 0)
-			(effects
-				(font

Commit message: Moving components around
Parts:
- removed D10: PMEG4005EJ, SparkFun-Semiconductor-Standard:SOD-323, symbol SparkFun-DiscreteSemi:D_Schottky_0.5A_40V_0.42V
- removed R46, R50: 33R, Resistor_SMD:R_0805_2012Metric, symbol Device:R
- added D10: PMEG4005EJ, SparkFun-Semiconductor-Standard:SOD-323, symbol Device:D_Schottky
- D3: footprint (none) -> Diode_SMD:D_SMC_Handsoldering
- D5: footprint (none) -> LED_SMD:LED_0805_2012Metric
Connections:
- net +3.3V: now also D10.2 (A)
- net at R57.2: now also D10.1 (K)
- no-connect marks 34 -> 35

Commit message: All components have been added
Parts:
- R23: footprint (none) -> Resistor_SMD:R_0805_2012Metric
- U3: footprint GNSS Board:SOIC127P599X175-8N -> gnss_board:SOIC127P599X175-8N
- U5: footprint RF_Module:ESP32-WROOM-32D -> RF_Module:ESP32-WROOM-32E
Changed lines of the file:
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@@
 	)
 	(junction
+		(at 92.71 120.65)
+		(diameter 0)
+		(color 0 0 0 0)
+	)
+	(junction
 		(at 339.09 232.41)
 		(diameter 0)
@@
 	)
 	(junction
-		(at 92.71 120.65)
-		(diameter 0)
-		(color 0 0 0 0)
-	)
-	(junction
 		(at 199.39 60.96)
 		(diameter 0)
@@
 	(wire
 		(pts
-			(xy 92.71 120.65) (xy 96.52 120.65)
+			(xy 320.04 91.44) (xy 325.12 91.44)
 		)
 		(stroke
@@
 	(wire
 		(pts
-			(xy 320.04 91.44) (xy 325.12 91.44)
+			(xy 350.52 49.53) (xy 350.52 48.26)
 		)
 		(stroke
@@
 	(wire
 		(pts
-			(xy 350.52 49.53) (xy 350.52 48.26)
+			(xy 255.27 255.27) (xy 255.27 256.54)
 		)
 		(stroke
@@
 	(wire
 		(pts
-			(xy 255.27 255.27) (xy 255.27 256.54)
+			(xy 92.71 120.65) (xy 96.52 120.65)
 		)
 		(stroke
@@
 			)
 		)
-		(property "Footprint" "GNSS Board:SOIC127P599X175-8N"
+		(property "Footprint" "gnss_board:SOIC127P599X175-8N"
 			(at 74.93 125.73 0)
 			(effects
@@
 			)
 		)
-		(property "Footprint" ""
+		(property "Footprint" "Resistor_SMD:R_0805_2012Metric"
 			(at 100.33 122.428 90)
 			(effects
@@
 			)
 		)
-		(property "Footprint" "RF_Module:ESP32-WROOM-32D"
+		(property "Footprint" "RF_Module:ESP32-WROOM-32E"
 			(at 110.49 260.35 0)
 			(effects

Commit message: Let's add this as well
Parts:
- added C29, C30, C31: 10uF, Capacitor_SMD:C_0805_2012Metric, symbol Device:C_Small
- added C32: 22uF, Capacitor_SMD:C_0805_2012Metric, symbol Device:C_Small
- added L4: FB0805, Inductor_SMD:L_0805_2012Metric_Pad1.15x1.40mm_HandSolder, symbol ESP32-PoE_Rev_L1:L
- C26: value 2.2uF -> 10uF
- J3: footprint SparkFun-Connector:U.FL -> Connector_Coaxial:U.FL_Molex_MCRF_73412-0110_Vertical
Connections:
- net +3.3V: now also C32.1, L4.2; no longer C26.2, C27.2, U6.33 (VCC), U6.34 (VCC)
- net GND: now also C29.1, C30.1, C31.1, C32.2
- net SW: now reaches C18.2, D3.1 (K), L2.1, R31.1, U4.1 (SW)
- new net VCC: C26.2, C27.2, C29.2, C30.2, C31.2, L4.1, U6.33 (VCC), U6.34 (VCC)
Other:
- moved on the sheet: C20, C27
